Commit message: Add SLAM integration, improve turning dynamics, and update documentation
- Add SLAM toolbox integration with configuration and launch files
- Improve front wheel turning: reduce friction (mu=0.001), increase slip (1.0), lower damping (0.001)
- Add friction to back wheels (mu=1.0) for better traction
- Lower center of mass for improved stability
- Increase caster mass and add pivot offset for better trailing
- Fix lidar frame_id conversion (Gazebo -> URDF frames)
- Update camera position to start at wheelchair
- Add comprehensive documentation:
  * SLAM_GUIDE.md - SLAM mapping instructions
  * DRIVING_GUIDE.md - Driving techniques for mapping
  * SPEED_SETTINGS.md - Speed parameter reference
  * NAV2_SETUP_GUIDE.md - Nav2 integration guide
- Update README.md with SLAM/Nav2 features and launch options
- Update requirements.txt with SLAM and Nav2 dependencies
- Clean up unwanted files (__pycache__, generated frames, zip files)
- Update .gitignore for maps directory

File: autonomous_wheelchair/src/wheelchair_description/urdf/wheelchair.urdf.xacro (robot description, xacro)
@@ -72,5 +72,5 @@
     <inertial>
       <mass value="${base_mass}"/>
-      <origin xyz="0.0 0.0 0.0" rpy="0.0 0.0 0.0"/>
+      <origin xyz="0.0 0.0 -0.05" rpy="0.0 0.0 0.0"/>  <!-- Lower CoM for better stability during turns -->
       <inertia
         ixx="${Ixx_val}" ixy="0.0" ixz="0.0"
@@ -159,4 +159,20 @@
           <cylinder length="${wheel_width_back}" radius="${wheel_radius_back}"/>
         </geometry>
+        <surface>
+          <friction>
+            <ode>
+              <mu>1.0</mu>     <!-- High friction for good grip (driving wheels) -->
+              <mu2>1.0</mu2>   <!-- High friction for good grip (driving wheels) -->
+              <slip1>0.0</slip1>  <!-- No slip for traction -->
+              <slip2>0.0</slip2>  <!-- No slip for traction -->
+            </ode>
+          </friction>
+          <contact>
+            <ode>
+              <kp>1000000.0</kp>
+              <kd>100.0</kd>
+            </ode>
+          </contact>
+        </surface>
       </collision>
     </link>
@@ -176,6 +192,6 @@
       <inertial>
         <origin xyz="0.0 0.0 0.0" rpy="0.0 0.0 0.0"/>
-        <mass value="0.2"/>
-        <inertia ixx="0.0001" ixy="0.0" ixz="0.0" iyy="0.0001" iyz="0.0" izz="0.0001"/>
+        <mass value="0.5"/>  <!-- Increased mass for better caster engagement -->
+        <inertia ixx="0.0005" ixy="0.0" ixz="0.0" iyy="0.0005" iyz="0.0" izz="0.0005"/>  <!-- Updated for increased mass -->
       </inertial>
       <visual name="${name}_caster_visual">
@@ -221,4 +237,21 @@
           <cylinder length="${wheel_width_front}" radius="${wheel_radius_front}"/>
         </geometry>
+        <surface>
+          <friction>
+            <ode>
+              <mu>0.001</mu>        <!-- Very low friction for easy lateral sliding -->
+              <mu2>0.001</mu2>      <!-- Very low friction for easy lateral sliding -->
+              <slip1>1.0</slip1>    <!-- Maximum slip for better turning -->
+              <slip2>1.0</slip2>    <!-- Maximum slip for better turning -->
+            </ode>
+          </friction>
+          <contact>
+            <ode>
+              <kp>1000000.0</kp>
+              <kd>100.0</kd>
+              <min_depth>0.001</min_depth>  <!-- Minimum contact depth -->
+            </ode>
+          </contact>
+        </surface>
       </collision>
     </link>
@@ -229,5 +262,5 @@
       <child link="${name}_caster_link"/>
       <axis xyz="0.0 0.0 1.0"/>
-      <dynamics damping="0.1" friction="0.0"/>
+      <dynamics damping="0.001" friction="0.0"/>  <!-- Very low damping for free caster rotation -->
       <limit effort="10.0" velocity="10.0"/>
     </joint>
@@ -235,9 +268,10 @@
     <joint name="${name}_joint" type="continuous">
       <!-- Place the wheel center below the caster mount by wheel_front_mount_height -->
-      <origin xyz="0.0 0.0 -${wheel_front_mount_height}" rpy="0.0 0.0 0.0"/>
+      <!-- Add 3cm forward offset to help caster trail naturally (improves turning) -->
+      <origin xyz="0.03 0.0 -${wheel_front_mount_height}" rpy="0.0 0.0 0.0"/>
       <parent link="${name}_caster_link"/>
       <child link="${name}_link"/>
       <axis xyz="0.0 1.0 0.0"/>
-      <dynamics damping="0.0" friction="0.0"/>
+      <dynamics damping="0.001" friction="0.0"/>  <!-- Very low damping for free wheel rotation -->
       <limit effort="50.0" velocity="50.0"/>
     </joint>
