Commit message: Fix: Add joint_state_publisher, fix camera stand position, add clock/joint_states bridges
- Added joint_state_publisher node to fix missing wheel transforms
- Fixed camera stand position (now touches base)
- Added /clock bridge for ROS time synchronization
- Added /joint_states bridge (with fallback to joint_state_publisher)
- Fixed robot_state_publisher remappings
- Fixed diff drive plugin filename (libignition-gazebo6-diff-drive-system.so)
- Updated camera and LiDAR positions to match new stand position

File: autonomous_wheelchair/src/wheelchair_description/urdf/wheelchair.gazebo.xacro (robot description, xacro)
@@ -20,4 +20,5 @@
     <material>Gazebo/Black</material>
   </gazebo>
+  <!-- wheel1_link: Back Right Wheel -->
   <gazebo reference="wheel1_link">
     <material>Gazebo/Black</material>
@@ -27,6 +28,7 @@
     <kd>100.0</kd>
     <minDepth>0.001</minDepth>
-    <maxDepth>0.15</maxDepth>
-  </gazebo>
+    <maxDepth>0.15</maxDepth>  <!-- Back wheel radius -->
+  </gazebo>
+  <!-- wheel2_link: Back Left Wheel -->
   <gazebo reference="wheel2_link">
     <material>Gazebo/Black</material>
@@ -36,6 +38,7 @@
     <kd>100.0</kd>
     <minDepth>0.001</minDepth>
-    <maxDepth>0.15</maxDepth>
-  </gazebo>
+    <maxDepth>0.15</maxDepth>  <!-- Back wheel radius -->
+  </gazebo>
+  <!-- wheel3_link: Front Right Wheel -->
   <gazebo reference="wheel3_link">
     <material>Gazebo/Black</material>
@@ -45,6 +48,7 @@
     <kd>100.0</kd>
     <minDepth>0.001</minDepth>
-    <maxDepth>0.095</maxDepth>
-  </gazebo>
+    <maxDepth>0.095</maxDepth>  <!-- Front wheel radius -->
+  </gazebo>
+  <!-- wheel4_link: Front Left Wheel -->
   <gazebo reference="wheel4_link">
     <material>Gazebo/Black</material>
@@ -54,31 +58,46 @@
     <kd>100.0</kd>
     <minDepth>0.001</minDepth>
-    <maxDepth>0.095</maxDepth>
+    <maxDepth>0.095</maxDepth>  <!-- Front wheel radius -->
   </gazebo>
   <gazebo reference="imu_sensor_link">
     <material>Gazebo/Blue</material>
   </gazebo>
-  <!-- ==================== DIRECT DIFF DRIVE PLUGIN - EXACT MATCH TO WORKING MODEL ==================== -->
+  <!-- ==================== DIRECT DIFF DRIVE PLUGIN ==================== -->
   <!--
-    Direct Gazebo diff drive plugin - EXACT same configuration as ros2-wheelchair-main
-    This matches the working implementation exactly for guaranteed compatibility
-    Configuration (matches working model exactly):
-    - left_joint: left_wheel_joint
-    - right_joint: right_wheel_joint
-    - wheel_separation: 2.6 (distance between wheel centers)
-    - wheel_radius: 0.8
-    - odom_publish_frequency: 10
-    - No explicit topic (uses default model/wheelchair/cmd_vel)
+    Direct Gazebo diff drive plugin for 4-wheel skid steer robot
+    Official Documentation Reference:
+    - Gazebo Fortress DiffDrive Plugin: https://gazebosim.org/api/gazebo/6/diff__drive_8hh.html
+    NOTE: The diff drive plugin only supports 2 joints (left and right).
+    For a 4-wheel robot, we use the back wheels as the primary drive wheels.
+    The front wheels will follow due to skid steer physics.
+    Configuration:
+    - left_joint: wheel2_joint (back left wheel)
+    - right_joint: wheel1_joint (back right wheel)
+    - wheel_separation: 0.52 (lateral distance between left and right wheel centers in meters)
+    - wheel_radius: 0.15 (back wheel radius in meters - using back wheels for drive)
+    - odom_publish_frequency: 10 Hz
+    - odom_frame_id: odom (ROS standard odometry frame)
+    - robot_base_frame: chassis (base frame name, matches URDF)
+    Topic Configuration:
+    - cmd_vel: Uses default Gazebo topic (model/wheelchair/cmd_vel)
+    - odometry: Uses default Gazebo topic (model/wheelchair/odometry)
+    These are bridged to ROS topics via ros_gz_bridge in launch file.
   -->
   <gazebo>
-    <plugin filename="libignition-gazebo-diff-drive-system.so"
+    <plugin filename="libignition-gazebo6-diff-drive-system.so"
             name="ignition::gazebo::systems::DiffDrive">
-      <left_joint>left_wheel_joint</left_joint>
-      <right_joint>right_wheel_joint</right_joint>
-      <wheel_separation>2.6</wheel_separation>
-      <wheel_radius>0.8</wheel_radius>
+      <left_joint>wheel2_joint</left_joint>      <!-- Back left wheel -->
+      <right_joint>wheel1_joint</right_joint>    <!-- Back right wheel -->
+      <wheel_separation>0.52</wheel_separation>  <!-- Lateral separation (m) -->
+      <wheel_radius>0.15</wheel_radius>         <!-- Back wheel radius (m) -->
       <odom_publish_frequency>10</odom_publish_frequency>
-      <!-- Topic commented out - uses default model/autonomous_wheelchair/cmd_vel -->
-      <!-- <topic>cmd_vel</topic> -->
+      <odom_frame_id>odom</odom_frame_id>        <!-- Odometry frame (ROS standard) -->
+      <robot_base_frame>chassis</robot_base_frame>  <!-- Base frame (matches URDF) -->
+      <!--
+        Note: cmd_vel and odometry topics use default Gazebo naming:
+        - cmd_vel: model/wheelchair/cmd_vel
+        - odometry: model/wheelchair/odometry
+        These are bridged to ROS topics in the launch file.
+      -->
     </plugin>
   </gazebo>
@@ -148,6 +167,6 @@
       </imu>
       <!-- plugin: explicit IMU system plugin (filename must match your installation) -->
-      <!-- Note: Plugin filename verified to exist: libignition-gazebo-imu-system.so -->
-      <plugin filename="ignition-gazebo-imu-system" name="gz::sim::systems::Imu">
+      <!-- For Gazebo Fortress, use the library filename with .so extension -->
+      <plugin filename="libignition-gazebo-imu-system.so" name="gz::sim::systems::Imu">
         <topic>/wheelchair/imu</topic>
         <frame_id>imu_sensor_link</frame_id>
@@ -242,32 +261,3 @@
     </sensor>
   </gazebo>
-  <!-- If you want GPU variant later, keep the original but comment it out while debugging:
-  <gazebo reference="base_laser">
-    <sensor name="lidar_gpu" type="gpu_lidar">
-      <always_on>true</always_on>
-      <update_rate>40</update_rate>
-      <visualize>true</visualize>
-      <lidar>
-        <scan>
-          <horizontal>
-            <samples>720</samples>
-            <resolution>1</resolution>
-            <min_angle>-3.14159265</min_angle>
-            <max_angle>3.14159265</max_angle>
-          </horizontal>
-        </scan>
-        <range>
-          <min>0.1</min>
-          <max>10.0</max>
-          <resolution>0.01</resolution>
-        </range>
-        <noise>
-          <type>gaussian</type>
-          <mean>0.0</mean>
-          <stddev>0.01</stddev>
-        </noise>
-      </lidar>
-    </sensor>
-  </gazebo>
-  -->
 </robot>

File: autonomous_wheelchair/src/wheelchair_description/urdf/wheelchair.ros2_control.xacro (robot description, xacro)
@@ -7,8 +7,11 @@
   -->
   <!-- ==================== ROS 2 CONTROL PARAMETERS ==================== -->
-  <xacro:property name="wheel_separation" value="0.52"/>  <!-- Distance between left and right wheel centers (m) -->
-  <xacro:property name="wheel_radius" value="0.15"/>      <!-- Wheel radius (m) - using back wheel radius -->
-  <xacro:property name="max_velocity" value="1.0"/>       <!-- Maximum linear velocity (m/s) -->
-  <xacro:property name="max_angular_velocity" value="2.0"/> <!-- Maximum angular velocity (rad/s) -->
+  <!-- Consistent with URDF parameters -->
+  <xacro:property name="wheel_separation" value="0.52"/>      <!-- Lateral separation between left and right wheels (m) -->
+  <xacro:property name="wheel_radius" value="0.15"/>            <!-- Back wheel radius (m) - primary drive wheels -->
+  <xacro:property name="max_linear_velocity" value="1.0"/>          <!-- Maximum linear velocity (m/s) -->
+  <xacro:property name="max_angular_velocity" value="2.0"/>   <!-- Maximum angular velocity (rad/s) -->
+  <!-- Maximum wheel angular velocity: v = ω * r, so ω = v / r = 1.0 / 0.15 = 6.67 rad/s -->
+  <xacro:property name="max_wheel_angular_velocity" value="6.67"/>  <!-- Max wheel angular velocity (rad/s) -->
   <!-- ==================== ROS 2 CONTROL HARDWARE INTERFACE ==================== -->
   <!--
@@ -24,45 +27,47 @@
     <!-- ==================== WHEEL JOINTS ==================== -->
     <!--
-      Joint naming convention:
-      - wheel1_joint: Back right wheel
-      - wheel2_joint: Back left wheel
-      - wheel3_joint: Front right wheel
-      - wheel4_joint: Front left wheel
+      Consistent joint naming convention (matches URDF):
+      - wheel1_joint: back_right_wheel (back right)
+      - wheel2_joint: back_left_wheel  (back left)
+      - wheel3_joint: front_right_wheel (front right)
+      - wheel4_joint: front_left_wheel  (front left)
       Controller mapping (from controllers.yaml):
-      - Left wheels: wheel2_joint, wheel4_joint
-      - Right wheels: wheel1_joint, wheel3_joint
+      - Left side wheels: wheel2_joint (back left), wheel4_joint (front left)
+      - Right side wheels: wheel1_joint (back right), wheel3_joint (front right)
     -->
-    <!-- Wheel 1: Back Right -->
+    <!-- wheel1_joint: Back Right Wheel -->
+    <!-- Note: Joint velocity interface uses angular velocity (rad/s), not linear velocity (m/s) -->
+    <!-- Max angular velocity = max_linear_velocity / wheel_radius = 1.0 / 0.15 = 6.67 rad/s -->
     <joint name="wheel1_joint">
       <command_interface name="velocity">
-        <param name="min">-${max_velocity}</param>
-        <param name="max">${max_velocity}</param>
+        <param name="min">-${max_wheel_angular_velocity}</param>
+        <param name="max">${max_wheel_angular_velocity}</param>
       </command_interface>
       <state_interface name="velocity"/>
       <state_interface name="position"/>
     </joint>
-    <!-- Wheel 2: Back Left -->
+    <!-- wheel2_joint: Back Left Wheel -->
     <joint name="wheel2_joint">
       <command_interface name="velocity">
-        <param name="min">-${max_velocity}</param>
-        <param name="max">${max_velocity}</param>
+        <param name="min">-${max_wheel_angular_velocity}</param>
+        <param name="max">${max_wheel_angular_velocity}</param>
       </command_interface>
       <state_interface name="velocity"/>
       <state_interface name="position"/>
     </joint>
-    <!-- Wheel 3: Front Right -->
+    <!-- wheel3_joint: Front Right Wheel -->
     <joint name="wheel3_joint">
       <command_interface name="velocity">
-        <param name="min">-${max_velocity}</param>
-        <param name="max">${max_velocity}</param>
+        <param name="min">-${max_wheel_angular_velocity}</param>
+        <param name="max">${max_wheel_angular_velocity}</param>
       </command_interface>
       <state_interface name="velocity"/>
       <state_interface name="position"/>
     </joint>
-    <!-- Wheel 4: Front Left -->
+    <!-- wheel4_joint: Front Left Wheel -->
     <joint name="wheel4_joint">
       <command_interface name="velocity">
-        <param name="min">-${max_velocity}</param>
-        <param name="max">${max_velocity}</param>
+        <param name="min">-${max_wheel_angular_velocity}</param>
+        <param name="max">${max_wheel_angular_velocity}</param>
       </command_interface>
       <state_interface name="velocity"/>

File: autonomous_wheelchair/src/wheelchair_description/urdf/wheelchair.urdf.xacro (robot description, xacro)
@@ -13,22 +13,26 @@
   <!-- Computed box inertial for chassis -->
   <!-- For box: I = m/12 * (dim1² + dim2²) -->
-  <!-- h² = 0.035² = 0.001225, w² = 0.44² = 0.1936, l² = 0.5² = 0.25 -->
-  <!-- Ixx = (10/12) * (0.001225 + 0.1936) = 0.16235416666666666 -->
-  <!-- Iyy = (10/12) * (0.25 + 0.001225) = 0.20935416666666665 -->
+  <!-- h = 0.05, w = 0.44, l = 0.5, m = 10.0 -->
+  <!-- h² = 0.05² = 0.0025, w² = 0.44² = 0.1936, l² = 0.5² = 0.25 -->
+  <!-- Ixx = (10/12) * (0.0025 + 0.1936) = 0.16341666666666668 -->
+  <!-- Iyy = (10/12) * (0.25 + 0.0025) = 0.21041666666666667 -->
   <!-- Izz = (10/12) * (0.25 + 0.1936) = 0.3696666666666667 -->
-  <xacro:property name="Ixx_val" value="0.16235416666666666"/>
-  <xacro:property name="Iyy_val" value="0.20935416666666665"/>
+  <xacro:property name="Ixx_val" value="0.16341666666666668"/>
+  <xacro:property name="Iyy_val" value="0.21041666666666667"/>
   <xacro:property name="Izz_val" value="0.3696666666666667"/>
-  <!-- Wheel parameters -->
-  <xacro:property name="wheel_radius_back" value="0.15"/>
-  <xacro:property name="wheel_width_back" value="0.04"/>
-  <xacro:property name="wheel_radius_front" value="0.095"/>
-  <xacro:property name="wheel_width_front" value="0.03"/>
-  <xacro:property name="wheel_mass" value="0.5"/>
-  <!-- Wheel positions (relative to base_uplayer_link) -->
-  <xacro:property name="wheel_separation_x" value="0.5"/>  <!-- Distance between front and back wheels -->
-  <xacro:property name="wheel_separation_y" value="0.52"/>  <!-- Distance between left and right wheels -->
-  <xacro:property name="wheel_base_x" value="0.25"/>  <!-- Half of wheel_separation_x -->
-  <xacro:property name="wheel_base_y" value="0.26"/>  <!-- Half of wheel_separation_y -->
+  <!-- ==================== WHEEL PARAMETERS ==================== -->
+  <!-- Consistent naming: back/front refer to position, left/right refer to side -->
+  <xacro:property name="wheel_radius_back" value="0.15"/>      <!-- Back wheel radius (m) -->
+  <xacro:property name="wheel_width_back" value="0.04"/>        <!-- Back wheel width (m) -->
+  <xacro:property name="wheel_radius_front" value="0.095"/>     <!-- Front wheel radius (m) -->
+  <xacro:property name="wheel_width_front" value="0.03"/>      <!-- Front wheel width (m) -->
+  <xacro:property name="wheel_mass" value="0.5"/>                <!-- Wheel mass (kg) -->
+  <!-- Wheel separation distances (relative to base_uplayer_link) -->
+  <xacro:property name="wheel_separation_longitudinal" value="0.5"/>   <!-- Distance between front and back wheels (m) -->
+  <xacro:property name="wheel_separation_lateral" value="0.52"/>      <!-- Distance between left and right wheels (m) -->
+  <xacro:property name="wheel_base_x" value="0.25"/>                  <!-- Half of longitudinal separation (m) -->
+  <xacro:property name="wheel_base_y" value="0.26"/>                  <!-- Half of lateral separation (m) -->
+  <!-- For diff drive calculations: use lateral separation -->
+  <xacro:property name="wheel_separation" value="0.52"/>              <!-- Lateral separation for diff drive (m) -->
   <!-- Base link height offset -->
   <xacro:property name="base_height_offset" value="0.21"/>
@@ -63,5 +67,5 @@
   <link name="base_uplayer_link">
     <visual name="chassis_visual">
-      <origin xyz="0 0 0" rpy="0 0 0"/>
+      <origin xyz="0.0 0.0 0.0" rpy="0.0 0.0 0.0"/>
       <geometry>
         <box size="${base_length} ${base_width} ${base_height}"/>
@@ -73,5 +77,5 @@
     <inertial>
       <mass value="${base_mass}"/>
-      <origin xyz="0 0 0" rpy="0 0 0"/>
+      <origin xyz="0.0 0.0 0.0" rpy="0.0 0.0 0.0"/>
       <!-- Using computed box inertia values (same as chassis since same dimensions) -->
       <inertia
@@ -86,5 +90,5 @@
     </collision>
     <collision name="caster_collision">
-      <origin xyz="-0.2 0 -0.05" rpy="0 0 0"/>
+      <origin xyz="-0.2 0.0 -0.05" rpy="0.0 0.0 0.0"/>
       <geometry>
         <sphere radius="0.05"/>
@@ -102,5 +106,5 @@
     </collision>
     <visual name="caster_visual">
-      <origin xyz="0.0 0 -0.05" rpy="0 0 0"/>
+      <origin xyz="-0.2 0.0 -0.05" rpy="0.0 0.0 0.0"/>  <!-- Match collision position -->
       <geometry>
         <sphere radius="0.05"/>
@@ -127,5 +131,5 @@
       </inertial>
       <visual name="${name}_visual">
-        <origin xyz="0.0 0.0 0.0" rpy="1.570795 0.0 0.0"/>
+        <origin xyz="0.0 0.0 0.0" rpy="1.57079632679 0.0 0.0"/>  <!-- π/2 rotation for cylinder -->
         <geometry>
           <cylinder length="${wheel_width_back}" radius="${wheel_radius_back}"/>
@@ -136,5 +140,5 @@
       </visual>
       <collision name="${name}_collision">
-        <origin xyz="0.0 0.0 0.0" rpy="1.570795 0.0 0.0"/>
+        <origin xyz="0.0 0.0 0.0" rpy="1.57079632679 0.0 0.0"/>  <!-- π/2 rotation for cylinder -->
         <geometry>
           <cylinder length="${wheel_width_back}" radius="${wheel_radius_back}"/>
@@ -162,5 +166,5 @@
       </inertial>
       <visual name="${name}_visual">
-        <origin xyz="0.0 0.0 0.0" rpy="1.570795 0.0 0.0"/>
+        <origin xyz="0.0 0.0 0.0" rpy="1.57079632679 0.0 0.0"/>  <!-- π/2 rotation for cylinder -->
         <geometry>
           <cylinder length="${wheel_width_front}" radius="${wheel_radius_front}"/>
@@ -171,5 +175,5 @@
       </visual>
       <collision name="${name}_collision">
-        <origin xyz="0.0 0.0 0.0" rpy="1.570795 0.0 0.0"/>
+        <origin xyz="0.0 0.0 0.0" rpy="1.57079632679 0.0 0.0"/>  <!-- π/2 rotation for cylinder -->
         <geometry>
           <cylinder length="${wheel_width_front}" radius="${wheel_radius_front}"/>
@@ -184,17 +188,21 @@
     </joint>
   </xacro:macro>
-  <!-- Create wheels -->
-  <!-- Back right wheel (wheel1) -->
-  <xacro:wheel_back name="wheel1" x="-${wheel_base_x}" y="-${wheel_base_y}"/>
-  <!-- Back left wheel (wheel2) -->
-  <xacro:wheel_back name="wheel2" x="-${wheel_base_x}" y="${wheel_base_y}"/>
-  <!-- Front right wheel (wheel3) -->
-  <xacro:wheel_front name="wheel3" x="${wheel_base_x}" y="-${wheel_base_y}"/>
-  <!-- Front left wheel (wheel4) -->
-  <xacro:wheel_front name="wheel4" x="${wheel_base_x}" y="${wheel_base_y}"/>
+  <!-- ==================== WHEEL INSTANTIATION ==================== -->
+  <!-- Consistent naming convention:
+       - wheel1: back_right_wheel (back right)
+       - wheel2: back_left_wheel  (back left)
+       - wheel3: front_right_wheel (front right)
+       - wheel4: front_left_wheel  (front left)
+       Joint names: wheel1_joint, wheel2_joint, wheel3_joint, wheel4_joint
+       Link names: wheel1_link, wheel2_link, wheel3_link, wheel4_link
+  -->
+  <xacro:wheel_back name="wheel1" x="-${wheel_base_x}" y="-${wheel_base_y}"/>  <!-- Back Right -->
+  <xacro:wheel_back name="wheel2" x="-${wheel_base_x}" y="${wheel_base_y}"/>     <!-- Back Left -->
+  <xacro:wheel_front name="wheel3" x="${wheel_base_x}" y="-${wheel_base_y}"/>    <!-- Front Right -->
+  <xacro:wheel_front name="wheel4" x="${wheel_base_x}" y="${wheel_base_y}"/>    <!-- Front Left -->
   <!-- ==================== IMU SENSOR ==================== -->
   <link name="imu_sensor_link">
     <collision>
-      <origin xyz="0 0 0" rpy="0 0 0"/>
+      <origin xyz="0.0 0.0 0.0" rpy="0.0 0.0 0.0"/>
       <geometry>
         <box size="0.02 0.02 0.02"/>
@@ -202,5 +210,5 @@
     </collision>
     <visual>
-      <origin xyz="0 0 0" rpy="0 0 0"/>
+      <origin xyz="0.0 0.0 0.0" rpy="0.0 0.0 0.0"/>
       <geometry>
         <box size="0.02 0.02 0.02"/>
@@ -212,10 +220,9 @@
     <inertial>
       <mass value="0.001"/>
-      <origin xyz="0 0 0" rpy="0 0 0"/>
-      <inertia ixx="0.00000015" ixy="0" ixz="0" iyy="0.00000015" iyz="0" izz="0.00000015"/>
+      <origin xyz="0.0 0.0 0.0" rpy="0.0 0.0 0.0"/>
+      <inertia ixx="0.00000015" ixy="0.0" ixz="0.0" iyy="0.00000015" iyz="0.0" izz="0.00000015"/>
     </inertial>
   </link>
   <joint name="imu_sensor_joint" type="fixed">
-    <axis xyz="0 0 1"/>
     <origin xyz="0.0 0.0 0.23" rpy="0.0 0.0 0.0"/>
     <parent link="chassis"/>
@@ -246,5 +253,7 @@
   </link>
   <joint name="camera_stand_joint" type="fixed">
-    <origin xyz="-0.22 0.0 0.58" rpy="0.0 0.0 0.0"/>
+    <!-- Position: base top is at z=0.235m (0.21 + 0.025), stand center should be at base top + half stand height -->
+    <!-- Stand height = 0.435m, so center = 0.235 + 0.2175 = 0.4525m -->
+    <origin xyz="-0.22 0.0 0.4525" rpy="0.0 0.0 0.0"/>
     <parent link="chassis"/>
     <child link="camera_stand_link"/>
@@ -257,6 +266,6 @@
       <inertia ixx="0.01" ixy="0.0" ixz="0.0" iyy="0.01" iyz="0.0" izz="0.01"/>
     </inertial>
-    <visual name="camera_visual">
-      <origin xyz="0.0 0.00 0.03" rpy="0 0 0.0"/>
+      <visual name="camera_visual">
+      <origin xyz="0.0 0.0 0.03" rpy="0.0 0.0 0.0"/>
       <geometry>
         <box size="0.1 0.2 0.04"/>
@@ -267,5 +276,5 @@
     </visual>
     <collision>
-      <origin xyz="0.0 0.00 0.03" rpy="0 0 0.0"/>
+      <origin xyz="0.0 0.0 0.03" rpy="0.0 0.0 0.0"/>
       <geometry>
         <box size="0.1 0.2 0.04"/>
@@ -276,13 +285,20 @@
     <parent link="camera_stand_link"/>
     <child link="camera_link"/>
-    <origin xyz="0.0 0.0 0.21" rpy="0 0.0 0.0"/>
+    <!-- Camera at top of stand: stand center is at z=0.4525, stand extends to z=0.4525+0.2175=0.67 -->
+    <!-- Camera should be at top of stand, so position at stand top + half camera height -->
+    <!-- Camera height = 0.04m, so center = 0.67 + 0.02 = 0.69m from stand center -->
+    <!-- But wait, stand center is at 0.4525, stand top is at 0.4525+0.2175=0.67 -->
+    <!-- Camera center should be at stand top + half camera height = 0.67 + 0.02 = 0.69 -->
+    <!-- Relative to stand center: 0.69 - 0.4525 = 0.2375 -->
+    <origin xyz="0.0 0.0 0.2375" rpy="0.0 0.0 0.0"/>
   </joint>
   <!-- Kinect Optical Frame -->
   <joint name="kinect_optical_joint" type="fixed">
-    <origin xyz="0 0 0" rpy="-1.5707 0 -1.5707"/>
+    <origin xyz="0.0 0.0 0.0" rpy="-1.57079632679 0.0 -1.57079632679"/>  <!-- -π/2, 0, -π/2 -->
     <parent link="camera_link"/>
     <child link="kinect_optical"/>
   </joint>
   <link name="kinect_optical">
+    <!-- Kinect optical frame - minimal link for TF tree (no visual/collision needed) -->
     <inertial>
       <mass value="0.0001"/>
@@ -297,5 +313,5 @@
   <link name="base_laser">
     <visual>
-      <origin xyz="-0.015 0.00 0.015" rpy="0 0 0.0"/>
+      <origin xyz="0.0 0.0 0.0" rpy="0.0 0.0 0.0"/>  <!-- Aligned with collision -->
       <geometry>
         <cylinder length="0.05" radius="0.05"/>
@@ -313,6 +329,6 @@
     <inertial>
       <mass value="0.1"/>
-      <origin xyz="0 0 0" rpy="0 0 0"/>
-      <inertia ixx="1e-6" ixy="0" ixz="0" iyy="1e-6" iyz="0" izz="1e-6"/>
+      <origin xyz="0.0 0.0 0.0" rpy="0.0 0.0 0.0"/>
+      <inertia ixx="1e-6" ixy="0.0" ixz="0.0" iyy="1e-6" iyz="0.0" izz="1e-6"/>
     </inertial>
   </link>
@@ -320,7 +336,8 @@
     <parent link="chassis"/>
     <child link="base_laser"/>
-    <!-- Position: camera_stand is at (-0.22, 0.0, 0.58), lidar is at (0.015, 0.0, 0.18) relative to camera_stand -->
-    <!-- So lidar absolute position: (-0.22+0.015, 0.0, 0.58+0.18) = (-0.205, 0.0, 0.76) -->
-    <origin xyz="-0.205 0.0 0.76" rpy="0.0 0.0 0.0"/>
+    <!-- Position: camera_stand center is now at (-0.22, 0.0, 0.4525) -->
+    <!-- Camera is at top of stand: z = 0.4525 + 0.2175 (stand half-height) + 0.2375 (camera offset) = 0.9075 -->
+    <!-- Lidar should be near camera, adjusted position -->
+    <origin xyz="-0.205 0.0 0.9075" rpy="0.0 0.0 0.0"/>
   </joint>
   <!-- ==================== STRUCTURAL COMPONENTS (simplified) ==================== -->
