Commit message: Cleanup docs and update launch instructions

File: autonomous_wheelchair/src/wheelchair_description/urdf/wheelchair.gazebo.xacro (robot description, xacro)
@@ -91,13 +91,10 @@
       <wheel_separation>0.52</wheel_separation>  <!-- Lateral separation (m) -->
       <wheel_radius>0.15</wheel_radius>         <!-- Back wheel radius (m) -->
-      <odom_publish_frequency>10</odom_publish_frequency>
+      <odom_publish_frequency>5</odom_publish_frequency>  <!-- Reduced from 10 to 5 Hz for better performance -->
       <odom_frame_id>odom</odom_frame_id>        <!-- Odometry frame (ROS standard) -->
-      <robot_base_frame>chassis</robot_base_frame>  <!-- Base frame (matches URDF) -->
-      <!--
-        Note: cmd_vel and odometry topics use default Gazebo naming:
-        - cmd_vel: model/wheelchair/cmd_vel
-        - odometry: model/wheelchair/odometry
-        These are bridged to ROS topics in the launch file.
-      -->
+      <robot_base_frame>base_uplayer_link</robot_base_frame>  <!-- Base frame where wheels are attached (not chassis) -->
+      <!-- Note: Plugin uses default topic naming: model/wheelchair/cmd_vel and model/wheelchair/odometry -->
+      <!-- These are automatically created based on model name "wheelchair" -->
+      <!-- No explicit topic parameter needed - plugin uses default naming convention -->
     </plugin>
   </gazebo>
@@ -116,9 +113,9 @@
   <!-- ==================== IMU SENSOR ==================== -->
   <!-- === IMU (explicit topic + frame_id + plugin) === -->
-  <gazebo reference="imu_sensor_link">
-    <sensor name="imu_sensor" type="imu">
-      <always_on>true</always_on>
-      <update_rate>100</update_rate>
-      <visualize>true</visualize>
+        <gazebo reference="imu_sensor_link">
+          <sensor name="imu_sensor" type="imu">
+            <always_on>true</always_on>
+            <update_rate>30</update_rate>  <!-- Reduced from 100 to 30 Hz for better performance -->
+            <visualize>false</visualize>  <!-- Disabled visualization to reduce lag -->
       <!-- explicit ros topic name and frame id to avoid auto-path surprises -->
       <topic>/wheelchair/imu</topic>
@@ -176,19 +173,19 @@
   <!-- ==================== RGB CAMERA ==================== -->
   <!-- === RGB Camera (namespaced topic, explicit frame id) === -->
-  <gazebo reference="camera_link">
-    <sensor name="camera_rgb" type="camera">
-      <always_on>true</always_on>
-      <update_rate>30</update_rate>
-      <visualize>true</visualize>
-      <!-- explicit namespaced topic and frame -->
-      <topic>/wheelchair/camera/image_raw</topic>
-      <frame_id>camera_link</frame_id>
-      <camera name="camera">
-        <horizontal_fov>1.047</horizontal_fov>
-        <image>
-          <width>640</width>
-          <height>480</height>
-          <format>R8G8B8</format>
-        </image>
+        <gazebo reference="camera_link">
+          <sensor name="camera_rgb" type="camera">
+            <always_on>true</always_on>
+            <update_rate>10</update_rate>  <!-- Reduced from 30 to 10 Hz for better performance -->
+            <visualize>false</visualize>  <!-- Disabled visualization to reduce lag -->
+            <!-- explicit namespaced topic and frame -->
+            <topic>/wheelchair/camera/image_raw</topic>
+            <frame_id>camera_link</frame_id>
+            <camera name="camera">
+              <horizontal_fov>1.047</horizontal_fov>
+              <image>
+                <width>320</width>  <!-- Reduced from 640 to 320 for better performance -->
+                <height>240</height>  <!-- Reduced from 480 to 240 for better performance -->
+                <format>R8G8B8</format>
+              </image>
         <clip>
           <near>0.1</near>
@@ -202,17 +199,17 @@
   <!-- ==================== DEPTH CAMERA ==================== -->
   <!-- === Depth Camera (namespaced topics) === -->
-  <gazebo reference="camera_link">
-    <sensor name="depth_camera" type="depth_camera">
-      <always_on>true</always_on>
-      <update_rate>30</update_rate>
-      <visualize>true</visualize>
-      <topic>/wheelchair/camera/depth</topic>
-      <frame_id>camera_link</frame_id>
-      <camera name="depth_camera">
-        <image>
-          <width>640</width>
-          <height>480</height>
-          <format>R_FLOAT32</format>
-        </image>
+        <gazebo reference="camera_link">
+          <sensor name="depth_camera" type="depth_camera">
+            <always_on>true</always_on>
+            <update_rate>10</update_rate>  <!-- Reduced from 30 to 10 Hz for better performance -->
+            <visualize>false</visualize>  <!-- Disabled visualization to reduce lag -->
+            <topic>/wheelchair/camera/depth</topic>
+            <frame_id>camera_link</frame_id>
+            <camera name="depth_camera">
+              <image>
+                <width>320</width>  <!-- Reduced from 640 to 320 for better performance -->
+                <height>240</height>  <!-- Reduced from 480 to 240 for better performance -->
+                <format>R_FLOAT32</format>
+              </image>
         <clip>
           <near>0.1</near>
@@ -229,26 +226,26 @@
   <!-- ==================== LIDAR SENSOR ==================== -->
   <!-- === GPU LIDAR (for RTX GPU systems) === -->
-  <gazebo reference="base_laser">
-    <sensor name="lidar" type="gpu_lidar">
-      <always_on>true</always_on>
-      <update_rate>40</update_rate>
-      <visualize>true</visualize>
-      <!-- namespaced topic - easier for bridge mapping -->
-      <topic>/wheelchair/scan</topic>
-      <frame_id>base_laser</frame_id>
-      <lidar>
-        <scan>
-          <horizontal>
-            <samples>360</samples>          <!-- reduce from 720 to reduce load while debugging -->
-            <resolution>1</resolution>
-            <min_angle>-3.14159</min_angle>
-            <max_angle>3.14159</max_angle>
-          </horizontal>
-        </scan>
-        <range>
-          <min>0.1</min>
-          <max>10.0</max>
-          <resolution>0.01</resolution>
-        </range>
+        <gazebo reference="base_laser">
+          <sensor name="lidar" type="gpu_lidar">
+            <always_on>true</always_on>
+            <update_rate>10</update_rate>  <!-- Reduced from 40 to 10 Hz for better performance -->
+            <visualize>false</visualize>  <!-- Disabled visualization to reduce lag -->
+            <!-- namespaced topic - easier for bridge mapping -->
+            <topic>/wheelchair/scan</topic>
+            <frame_id>base_laser</frame_id>
+            <lidar>
+              <scan>
+                <horizontal>
+                  <samples>180</samples>  <!-- Reduced from 360 to 180 for better performance -->
+                  <resolution>1</resolution>
+                  <min_angle>-3.14159</min_angle>
+                  <max_angle>3.14159</max_angle>
+                </horizontal>
+              </scan>
+              <range>
+                <min>0.1</min>
+                <max>10.0</max>
+                <resolution>0.05</resolution>  <!-- Reduced from 0.01 to 0.05 for better performance -->
+              </range>
         <noise>
           <type>gaussian</type>

File: autonomous_wheelchair/src/wheelchair_description/urdf/wheelchair.urdf.xacro (robot description, xacro)
@@ -147,5 +147,7 @@
     </link>
     <joint name="${name}_joint" type="continuous">
-      <origin xyz="${x} ${y} 0.0" rpy="0.0 0.0 0.0"/>
+      <!-- Wheel center should be at negative wheel radius below base_uplayer_link center -->
+      <!-- This positions the wheel so it touches the ground -->
+      <origin xyz="${x} ${y} -${wheel_radius_back}" rpy="0.0 0.0 0.0"/>
       <parent link="base_uplayer_link"/>
       <child link="${name}_link"/>
@@ -182,5 +184,7 @@
     </link>
     <joint name="${name}_joint" type="continuous">
-      <origin xyz="${x} ${y} 0.0" rpy="0.0 0.0 0.0"/>
+      <!-- Wheel center should be at negative wheel radius below base_uplayer_link center -->
+      <!-- Front wheels have smaller radius, so less negative z -->
+      <origin xyz="${x} ${y} -${wheel_radius_front}" rpy="0.0 0.0 0.0"/>
       <parent link="base_uplayer_link"/>
       <child link="${name}_link"/>

Commit message: Clean up codebase for ROS 2 Humble and Gazebo Fortress
- Fixed Gazebo Fortress plugin naming (ignition::gazebo -> gz::sim)
- Fixed view_robot_rviz2.launch.py to avoid duplicate robot_state_publisher
- Removed debug scripts (debug_turning.sh, launch_rviz_debug.sh)
- Cleaned trailing whitespace in package.xml and CMakeLists.txt
- Updated front wheels to caster configuration for proper rotation
- Adjusted front wheel friction parameters for better skid-steer behavior
- Updated spawn height calculation for proper wheel-ground contact
- Removed unused dependencies from package.xml

File: autonomous_wheelchair/src/wheelchair_description/urdf/wheelchair.gazebo.xacro (robot description, xacro)
@@ -86,5 +86,5 @@
   <gazebo>
     <plugin filename="libignition-gazebo6-diff-drive-system.so"
-            name="ignition::gazebo::systems::DiffDrive">
+            name="gz::sim::systems::DiffDrive">
       <left_joint>wheel2_joint</left_joint>      <!-- Back left wheel -->
       <right_joint>wheel1_joint</right_joint>    <!-- Back right wheel -->

File: autonomous_wheelchair/src/wheelchair_description/urdf/wheelchair.urdf.xacro (robot description, xacro)
@@ -28,4 +28,19 @@
   <xacro:property name="wheel_width_front" value="0.03"/>      <!-- Front wheel width (m) -->
   <xacro:property name="wheel_mass" value="0.5"/>                <!-- Wheel mass (kg) -->
+  <!--
+    Front wheel mount drop (distance from base_uplayer_link origin down to front wheel center).
+    We pick this so that both front and back wheels touch the ground with the SAME spawn z.
+    Back wheel bottom z:
+      z_bottom_back = z_spawn + base_height_offset - 2 * wheel_radius_back
+    For wheels to touch ground: z_bottom_back = 0  =>  z_spawn = 2*R_back - base_height_offset
+      With R_back = 0.15, base_height_offset = 0.21:  z_spawn = 0.30 - 0.21 = 0.09 m
+    For the front wheel (radius R_front) at the same z_spawn, we want:
+      z_bottom_front = z_spawn + base_height_offset - wheel_front_mount_height - R_front = 0
+      => wheel_front_mount_height = z_spawn + base_height_offset - R_front
+      = 0.09 + 0.21 - 0.095 = 0.205 m
+    So the front wheel center hangs 0.205 m below the base origin, and the wheel radius
+    is 0.095 m, giving an 11 cm “metal fork” / spacer which visually raises the chair front.
+  -->
+  <xacro:property name="wheel_front_mount_height" value="0.205"/>
   <!-- Wheel separation distances (relative to base_uplayer_link) -->
   <xacro:property name="wheel_separation_longitudinal" value="0.5"/>   <!-- Distance between front and back wheels (m) -->
@@ -155,6 +170,31 @@
     </joint>
   </xacro:macro>
-  <!-- Wheel macro for front wheels -->
+  <!-- Wheel macro for front wheels (modeled as casters: yaw joint + wheel roll joint) -->
   <xacro:macro name="wheel_front" params="name x y">
+    <!-- Caster mount link (small metal fork under the base) -->
+    <link name="${name}_caster_link">
+      <inertial>
+        <origin xyz="0.0 0.0 0.0" rpy="0.0 0.0 0.0"/>
+        <mass value="0.2"/>
+        <inertia ixx="0.0001" ixy="0.0" ixz="0.0" iyy="0.0001" iyz="0.0" izz="0.0001"/>
+      </inertial>
+      <visual name="${name}_caster_visual">
+        <!-- Simple vertical bar representing the metal support -->
+        <origin xyz="0.0 0.0 -${wheel_front_mount_height * 0.5}" rpy="0.0 0.0 0.0"/>
+        <geometry>
+          <box size="0.02 0.02 ${wheel_front_mount_height}"/>
+        </geometry>
+        <material name="gray">
+          <color rgba="0.5 0.5 0.5 1.0"/>
+        </material>
+      </visual>
+      <collision name="${name}_caster_collision">
+        <origin xyz="0.0 0.0 -${wheel_front_mount_height * 0.5}" rpy="0.0 0.0 0.0"/>
+        <geometry>
+          <box size="0.02 0.02 ${wheel_front_mount_height}"/>
+        </geometry>
+      </collision>
+    </link>
+    <!-- Wheel link (same as before, attached to caster link instead of base) -->
     <link name="${name}_link">
       <inertial>
@@ -183,11 +223,22 @@
       </collision>
     </link>
+    <!-- Caster yaw joint: base -> caster link (rotation about Z) -->
+    <joint name="${name}_caster_yaw_joint" type="continuous">
+      <origin xyz="${x} ${y} 0.0" rpy="0.0 0.0 0.0"/>
+      <parent link="base_uplayer_link"/>
+      <child link="${name}_caster_link"/>
+      <axis xyz="0.0 0.0 1.0"/>
+      <dynamics damping="0.1" friction="0.0"/>
+      <limit effort="10.0" velocity="10.0"/>
+    </joint>
+    <!-- Wheel roll joint: caster link -> wheel (rotation about Y) -->
     <joint name="${name}_joint" type="continuous">
-      <!-- Wheel center should be at negative wheel radius below base_uplayer_link center -->
-      <!-- Front wheels have smaller radius, so less negative z -->
-      <origin xyz="${x} ${y} -${wheel_radius_front}" rpy="0.0 0.0 0.0"/>
-      <parent link="base_uplayer_link"/>
+      <!-- Place the wheel center below the caster mount by wheel_front_mount_height -->
+      <origin xyz="0.0 0.0 -${wheel_front_mount_height}" rpy="0.0 0.0 0.0"/>
+      <parent link="${name}_caster_link"/>
       <child link="${name}_link"/>
       <axis xyz="0.0 1.0 0.0"/>
+      <dynamics damping="0.0" friction="0.0"/>
+      <limit effort="50.0" velocity="50.0"/>
     </joint>
   </xacro:macro>

Commit message: Update wheelchair model: lidar on back bar, Nav2 readiness, and improvements
- Move lidar sensor to back bar to prevent self-detection
- Add Nav2 readiness checker script and documentation
- Implement odom_to_tf node for proper TF tree
- Add lidar self-filtering node
- Update front wheels with caster mechanism
- Optimize contact parameters for realistic dynamics
- Update README with latest features
- Update requirements.txt with all dependencies
- Clean up unwanted files (CALCULATE_NEW_COM.md, generated frames)
- Add helper scripts for Nav2 integration

File: autonomous_wheelchair/src/wheelchair_description/urdf/wheelchair.gazebo.xacro (robot description, xacro)
@@ -91,5 +91,5 @@
       <wheel_separation>0.52</wheel_separation>  <!-- Lateral separation (m) -->
       <wheel_radius>0.15</wheel_radius>         <!-- Back wheel radius (m) -->
-      <odom_publish_frequency>5</odom_publish_frequency>  <!-- Reduced from 10 to 5 Hz for better performance -->
+      <odom_publish_frequency>10</odom_publish_frequency>  <!-- 10 Hz - balanced rate for RViz -->
       <odom_frame_id>odom</odom_frame_id>        <!-- Odometry frame (ROS standard) -->
       <robot_base_frame>base_uplayer_link</robot_base_frame>  <!-- Base frame where wheels are attached (not chassis) -->
@@ -234,4 +234,24 @@
             <topic>/wheelchair/scan</topic>
             <frame_id>base_laser</frame_id>
+            <!-- Ignore robot's own links to prevent self-detection -->
+            <!-- Note: Lidar is mounted on back_link, so back_link is ignored to prevent seeing the mounting surface -->
+            <ignore>
+              <link>chassis</link>
+              <link>base_uplayer_link</link>
+              <link>base_link</link>
+              <link>seat_link</link>
+              <link>back_link</link>  <!-- Back bar where lidar is mounted -->
+              <link>base_laser</link>  <!-- Ignore lidar itself -->
+              <link>camera_stand_link</link>
+              <link>camera_link</link>
+              <link>kinect_optical</link>
+              <link>imu_sensor_link</link>
+              <link>wheel1_link</link>
+              <link>wheel2_link</link>
+              <link>wheel3_link</link>
+              <link>wheel4_link</link>
+              <link>wheel3_caster_link</link>
+              <link>wheel4_caster_link</link>
+            </ignore>
             <lidar>
               <scan>

File: autonomous_wheelchair/src/wheelchair_description/urdf/wheelchair.urdf.xacro (robot description, xacro)
@@ -389,10 +389,12 @@
   </link>
   <joint name="base_link_to_lidar" type="fixed">
-    <parent link="chassis"/>
+    <parent link="back_link"/>
     <child link="base_laser"/>
-    <!-- Position: camera_stand center is now at (-0.22, 0.0, 0.4525) -->
-    <!-- Camera is at top of stand: z = 0.4525 + 0.2175 (stand half-height) + 0.2375 (camera offset) = 0.9075 -->
-    <!-- Lidar should be near camera, adjusted position -->
-    <origin xyz="-0.205 0.0 0.9075" rpy="0.0 0.0 0.0"/>
+    <!-- Position: Lidar mounted on back bar at lower height -->
+    <!-- Back bar is a box: 0.04 x 0.41 x 0.41 (width x height x depth) -->
+    <!-- Back bar center is at z=0, extends from z=-0.205 to z=+0.205 -->
+    <!-- Place lidar at lower position: z = 0.0 (center height) for better obstacle detection -->
+    <!-- Position slightly forward (x positive) to clear the back bar surface -->
+    <origin xyz="0.02 0.0 0.0" rpy="0.0 0.0 0.0"/>
   </joint>
   <!-- ==================== STRUCTURAL COMPONENTS (simplified) ==================== -->

Commit message: website+depthcamera+multisource cost map

File: autonomous_wheelchair/src/wheelchair_description/urdf/wheelchair.gazebo.xacro (robot description, xacro)
@@ -206,4 +206,5 @@
             <topic>/wheelchair/camera/depth</topic>
             <frame_id>camera_link</frame_id>
+            <gz_frame_id>camera_link</gz_frame_id> <!-- Gazebo frame id -->
             <camera name="depth_camera">
               <image>

File: autonomous_wheelchair/src/wheelchair_description/urdf/wheelchair.urdf.xacro (robot description, xacro)
@@ -380,5 +380,5 @@
     <!-- Camera center should be at stand top + half camera height = 0.67 + 0.02 = 0.69 -->
     <!-- Relative to stand center: 0.69 - 0.4525 = 0.2375 -->
-    <origin xyz="0.0 0.0 0.2375" rpy="0.0 0.0 0.0"/>
+    <origin xyz="0.0 0.0 0.2375" rpy="0.0 0.2618 0.0"/>
   </joint>
   <!-- Kinect Optical Frame -->
